File: ai03-tutorial.sch (KiCad schematic (older format))
At the start: 24 parts, among them SW1 SW_Push, U1 ATmega32U4-AU, Y1 16MHz

Commit message: pcb mostly done
Parts:
- MX1, MX2, MX3, MX4: footprint (none) -> MX_Alps_Hybrid:MX-1U-NoLED
Changed lines of the file:
@@
 F 0 "MX1" H 1533 4223 60  0000 C CNN
 F 1 "MX-NoLED" H 1533 4149 20  0000 C CNN
-F 2 "" H 875 3975 60  0001 C CNN
+F 2 "MX_Alps_Hybrid:MX-1U-NoLED" H 875 3975 60  0001 C CNN
 F 3 "" H 875 3975 60  0001 C CNN
 	1    1500 4000
@@
 F 0 "MX2" H 2233 4223 60  0000 C CNN
 F 1 "MX-NoLED" H 2233 4149 20  0000 C CNN
-F 2 "" H 1575 3975 60  0001 C CNN
+F 2 "MX_Alps_Hybrid:MX-1U-NoLED" H 1575 3975 60  0001 C CNN
 F 3 "" H 1575 3975 60  0001 C CNN
 	1    2200 4000
@@
 F 0 "MX3" H 1533 4923 60  0000 C CNN
 F 1 "MX-NoLED" H 1533 4849 20  0000 C CNN
-F 2 "" H 875 4675 60  0001 C CNN
+F 2 "MX_Alps_Hybrid:MX-1U-NoLED" H 875 4675 60  0001 C CNN
 F 3 "" H 875 4675 60  0001 C CNN
 	1    1500 4700
@@
 F 0 "MX4" H 2233 4923 60  0000 C CNN
 F 1 "MX-NoLED" H 2233 4849 20  0000 C CNN
-F 2 "" H 1575 4675 60  0001 C CNN
+F 2 "MX_Alps_Hybrid:MX-1U-NoLED" H 1575 4675 60  0001 C CNN
 F 3 "" H 1575 4675 60  0001 C CNN
 	1    2200 4700
